File: 3V3_boost_regulator/3V3_boost_regulator.kicad_pcb (KiCad board)
At the start: 2 copper layers, 15.2 x 15.2 mm, 8 parts, among them J1 Input, J2 Output, U1 MCP1642B/D-33I

Commit message: Adjusted inductor pours
Routing:
- net GND: vias 0 -> 3
Changed lines of the file:
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@@
   (segment (start 163.83 106.9555) (end 161.5655 106.9555) (width 0.6) (layer "F.Cu") (net 3))
   (segment (start 164.8245 107.95) (end 166.37 107.95) (width 0.6) (layer "F.Cu") (net 3))
+  (via (at 171 104) (size 0.8) (drill 0.4) (layers "F.Cu" "B.Cu") (free) (net 3))
+  (via (at 169 99) (size 0.8) (drill 0.4) (layers "F.Cu" "B.Cu") (free) (net 3))
+  (via (at 166 99) (size 0.8) (drill 0.4) (layers "F.Cu" "B.Cu") (free) (net 3))
   (segment (start 164.084 111.252) (end 164.846 112.014) (width 0.3) (layer "F.Cu") (net 4))
   (segment (start 164.084 108.458) (end 164.084 111.252) (width 0.3) (layer "F.Cu") (net 4))
@@
   (segment (start 164.084 106.934) (end 161.29 104.14) (width 0.3) (layer "B.Cu") (net 4))
   (segment (start 167.12 105.63) (end 167.12 104.152) (width 0.3) (layer "F.Cu") (net 6))
-  (zone (net 4) (net_name "Net-(C1-Pad2)") (layer "F.Cu") (hatch edge 0.508)
+  (zone (net 3) (net_name "GND") (layers F&B.Cu) (name "GND") (hatch edge 0.508)
     (connect_pads yes (clearance 0.2))
     (min_thickness 0.3) (filled_areas_thickness no)
@@
     (polygon
       (pts
-        (xy 166.37 103.886)
-        (xy 165.354 103.886)
-        (xy 165.354 105.664)
-        (xy 160.02 105.664)
+        (xy 175.26 113.03)
+        (xy 160.02 113.03)
         (xy 160.02 97.79)
-        (xy 166.37 97.79)
+        (xy 175.26 97.79)
       )
     )
   )
-  (zone (net 1) (net_name "Net-(C2-Pad2)") (layer "F.Cu") (hatch edge 0.508)
+  (zone (net 4) (net_name "Net-(C1-Pad2)") (layer "F.Cu") (hatch edge 0.508)
+    (priority 2)
+    (connect_pads yes (clearance 0.2))
+    (min_thickness 0.3) (filled_areas_thickness no)
+    (fill yes (thermal_gap 0.3) (thermal_bridge_width 0.5) (smoothing fillet) (radius 0.5))
+    (polygon
+      (pts
+        (xy 165.77 103.64)
+        (xy 165.77 105.47)
+        (xy 163.94 105.47)
+        (xy 163.06 104.93)
+        (xy 163.63 99.8)
+        (xy 165.64 99.8)
+      )
+    )
+  )
+  (zone (net 1) (net_name "Net-(C2-Pad2)") (layer "F.Cu") (name "Vout") (hatch edge 0.508)
+    (priority 1)
     (connect_pads yes (clearance 0.2))
     (min_thickness 0.3) (filled_areas_thickness no)
@@
         (xy 175.26 110.744)
         (xy 170.18 110.744)
-        (xy 170.18 110.998)
         (xy 170.18 109.22)
         (xy 168.656 109.22)
@@
     )
   )
-  (zone (net 3) (net_name "GND") (layer "F.Cu") (hatch edge 0.508)
-    (priority 2)
+  (zone (net 3) (net_name "GND") (layer "F.Cu") (name "GND") (hatch edge 0.508)
     (connect_pads yes (clearance 0.2))
     (min_thickness 0.3) (filled_areas_thickness no)
@@
   )
   (zone (net 6) (net_name "Net-(L1-Pad2)") (layer "F.Cu") (hatch edge 0.508)
-    (priority 1)
+    (priority 2)
     (connect_pads yes (clearance 0.2))
     (min_thickness 0.3) (filled_areas_thickness no)
@@
     (polygon
       (pts
-        (xy 172.974 101.854)
-        (xy 170.942 103.886)
-        (xy 167.894 103.886)
-        (xy 167.386 104.394)
-        (xy 166.878 104.394)
-        (xy 166.37 103.886)
-        (xy 166.37 97.79)
-        (xy 172.974 97.79)
+        (xy 171.14 101.06)
+        (xy 171.14 102.53)
+        (xy 167.27 104.16)
+        (xy 167.27 104.48)
+        (xy 166.97 104.48)
+        (xy 166.97 103.56)
+        (xy 169.36 99.8)
+        (xy 171.14 99.8)
       )
     )
-  )
-  (zone (net 3) (net_name "GND") (layer "B.Cu") (hatch edge 0.508)
-    (connect_pads yes (clearance 0.2))
-    (min_thickness 0.3) (filled_areas_thickness no)
-    (fill yes (thermal_gap 0.3) (thermal_bridge_width 0.5) (smoothing fillet) (radius 0.5))
-    (polygon
-      (pts
-        (xy 175.26 113.03)
-        (xy 160.02 113.03)
-        (xy 160.02 97.79)
-        (xy 175.26 97.79)
-      )
-    )
